File: electronics/snowflake.brd (EAGLE design)
At the start: 43.7 x 37.8 mm, 49 parts, among them J1 USB-5PIN614105150721, J2 TC2030-SWD, Q1 FET-PSOT-23-3, U1 WS2812B, U10 WS2812B, U11 WS2812B, U12 WS2812B, U13 WS2812B, U2 WS2812B, U20 BMD-200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

Commit message: update readme
Parts:
- added VBUS: TARGET-PIN, firefly:TARGET-PIN-1MM
Connections:
- net N$14: now also VBUS.1
Changed lines of the file:
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@@
 <attribute name="NAME" x="11.501834375" y="-15.43681875" size="0.8128" layer="26" rot="MR120"/>
 </element>
+<element name="VBUS" library="firefly" package="TARGET-PIN-1MM" value="TARGET-PIN" x="-20.6" y="-25.1"/>
 </elements>
 <signals>
@@
 <wire x1="10.5" y1="-11.9" x2="6.1" y2="-11.9" width="0.5" layer="16"/>
 <via x="11.8" y="-9.5" extent="1-16" drill="0.3302"/>
+<contactref element="VBUS" pad="1"/>
+<wire x1="-0.777384375" y1="-17.1175" x2="-20.6" y2="-25.1" width="0" layer="19" extent="1-16"/>
 </signal>
 <signal name="SWDIO">

Commit message: misc tweaks
Parts:
- moved VBUS 41.2 mm to (14.7, -3.80)
- moved R6 0.45 mm to (15.5, -1.96)
- moved C19 0.22 mm to (18.2, -1.22)
- moved R1 0.22 mm to (13.5, -4.33)
Routing:
- net N$14: track 34.1 -> 37.3 mm
- net BATTERY_DIV_2: track 29.5 -> 30.2 mm
