File: electronics/snowflake.sch (EAGLE design)
At the start: 49 parts, among them J1 USB-5PIN614105150721, J2 TC2030-SWD, Q1 FET-PSOT-23-3, U1 WS2812B, U10 WS2812B, U11 WS2812B, U12 WS2812B, U13 WS2812B, U2 WS2812B, U20 BMD-200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

Commit message: update readme
Parts:
- added VBUS: TARGET-PIN, firefly:TARGET-PIN
Connections:
- net N$14: now also VBUS.1
Changed lines of the file:
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@@
 <part name="B-" library="firefly" deviceset="TARGET-PIN" device="WP-28AWG"/>
 <part name="V42" library="firefly" deviceset="GND" device=""/>
+<part name="VBUS" library="firefly" deviceset="TARGET-PIN" device=""/>
 </parts>
 <sheets>
@@
 <instance part="B-" gate="G$1" x="68.58" y="96.52" rot="R90"/>
 <instance part="V42" gate="GND" x="68.58" y="83.82"/>
+<instance part="VBUS" gate="G$1" x="25.4" y="83.82" rot="R90"/>
 </instances>
 <busses>
@@
 <wire x1="50.8" y1="73.66" x2="40.64" y2="73.66" width="0.1524" layer="91"/>
 <pinref part="C15" gate="G$1" pin="1"/>
-<wire x1="40.64" y1="73.66" x2="22.86" y2="73.66" width="0.1524" layer="91"/>
+<wire x1="40.64" y1="73.66" x2="25.4" y2="73.66" width="0.1524" layer="91"/>
+<wire x1="25.4" y1="73.66" x2="22.86" y2="73.66" width="0.1524" layer="91"/>
 <wire x1="40.64" y1="71.12" x2="40.64" y2="73.66" width="0.1524" layer="91"/>
 <junction x="40.64" y="73.66"/>
@@
 <junction x="40.64" y="109.22"/>
 <junction x="106.68" y="109.22"/>
-</segment>
-</net>
+<pinref part="VBUS" gate="G$1" pin="1"/>
+<wire x1="25.4" y1="76.2" x2="25.4" y2="73.66" width="0.1524" layer="91"/>
+<junction x="25.4" y="73.66"/>
+</segment>
+</net>
